Commit message: Upper Body Urdf Added

File: mobi_description/urdf/mobi.urdf.xacro (robot description, xacro)
@@ -5,3 +5,6 @@
     <xacro:include filename="$(find mobi_description)/urdf/ros2_control.xacro" />
     <xacro:include filename="$(find mobi_description)/urdf/mobi_base.xacro" />
+    <xacro:include filename="$(find mobi_description)/urdf/mobi_sensors.xacro" />
+    <xacro:include filename="$(find mobi_description)/urdf/mobi_rail.xacro" />
+    <xacro:include filename="$(find mobi_description)/urdf/mobi_head.xacro" />
 </robot>

File: mobi_description/urdf/mobi_base.xacro (robot description, xacro)
@@ -1,215 +1,134 @@
 <?xml version="1.0" ?>
 <robot name="mobi" xmlns:xacro="http://www.ros.org/wiki/xacro">
-<!-- Load Simulated or Real Hardware Interfaces -->
-<xacro:arg name="is_sim" default="true"/> <!-- Getting passed as false in hardware interface launch file-->
-<xacro:arg name="serial_port" default="/dev/ttyUSB0"/>
-<link name="base_footprint"/>
-<link name="base_link">
-    <inertial>
-        <origin xyz="0.0 0.0 -0.0" rpy="0.0 0.0 0.0"/>
-        <mass value="5.0"/>
-        <inertia ixx="0.1" ixy="0.0" ixz="0.0" iyy="0.1" iyz="0.0" izz="0.1"/>
-    </inertial>
-    <visual>
-        <origin xyz="0.0 0.0 -0.0" rpy="0.0 0.0 0.0"/>
-        <geometry>
-            <mesh filename="package://mobi_description/meshes/base_link.stl" scale="0.001 0.001 0.001"/>
-        </geometry>
-        <material name="silver"/>
-    </visual>
-    <collision>
-        <origin xyz="0.0 0.0 -0.0" rpy="0.0 0.0 0.0"/>
-        <geometry>
-             <mesh filename="package://mobi_description/meshes/base_link.stl" scale="0.001 0.001 0.001"/>
-        </geometry>
-    </collision>
-</link>
-<joint name="base_joint" type="fixed">
-    <origin xyz="0.0 0.0 0.0" rpy="0.0 0.0 0.0"/>
-    <parent link="base_footprint"/>
-    <child link="base_link"/>
-</joint>
-<link name="right_wheel">
-    <inertial>
-        <origin xyz="-0.17 0.175 -0.06" rpy="0.0 0.0 0.0"/>
-        <mass value="1.0"/>
-        <inertia ixx="0.1" ixy="0.0" ixz="0.0" iyy="0.1" iyz="0.0" izz="0.1"/>
-    </inertial>
-    <visual>
-        <origin xyz="-0.17 0.175 -0.06" rpy="0.0 0.0 0.0"/>
-        <geometry>
-            <mesh filename="package://mobi_description/meshes/right_wheel.stl" scale="0.001 0.001 0.001"/>
-        </geometry>
-        <material name="mud_yellow"/>
-    </visual>
-    <collision>
-        <origin xyz="-0.17 0.175 -0.06" rpy="0.0 0.0 0.0"/>
-        <geometry>
-             <mesh filename="package://mobi_description/meshes/right_wheel.stl" scale="0.001 0.001 0.001"/>
-        </geometry>
-    </collision>
-</link>
-<joint name="right_wheel_joint" type="continuous">
-    <origin xyz="0.17 -0.175 0.06" rpy="0.0 0.0 0.0"/>
-    <parent link="base_link"/>
-    <child link="right_wheel"/>
-    <axis xyz="-0.0 1.0 0.0"/>
-</joint>
-<link name="left_wheel">
-    <inertial>
-        <origin xyz="-0.169 -0.175 -0.059" rpy="0.0 0.0 0.0"/>
-        <mass value="1.0"/>
-        <inertia ixx="0.1" ixy="0.0" ixz="0.0" iyy="0.1" iyz="0.0" izz="0.1"/>
-    </inertial>
-    <visual>
-        <origin xyz="-0.169 -0.175 -0.059" rpy="0.0 0.0 0.0"/>
-        <geometry>
-            <mesh filename="package://mobi_description/meshes/left_wheel.stl" scale="0.001 0.001 0.001"/>
-        </geometry>
-        <material name="mud_yellow"/>
-    </visual>
-    <collision>
-        <origin xyz="-0.169 -0.175 -0.059" rpy="0.0 0.0 0.0"/>
-        <geometry>
-             <mesh filename="package://mobi_description/meshes/left_wheel.stl" scale="0.001 0.001 0.001"/>
-        </geometry>
-    </collision>
-</link>
-<joint name="left_wheel_joint" type="continuous">
-    <origin xyz="0.169 0.175 0.059" rpy="0.0 0.0 0.0"/>
-    <parent link="base_link"/>
-    <child link="left_wheel"/>
-    <axis xyz="-0.0 1.0 0.0"/>
-</joint>
-<link name="left_castor_wheel">
-    <inertial>
-        <origin xyz="0.23 -0.15 -0.08" rpy="0.0 0.0 0.0"/>
-        <mass value="1.0"/>
-        <inertia ixx="0.1" ixy="0.0" ixz="0.0" iyy="0.1" iyz="0.0" izz="0.1"/>
-    </inertial>
-    <visual>
-        <origin xyz="0.23 -0.15 -0.08" rpy="0.0 0.0 0.0"/>
-        <geometry>
-            <mesh filename="package://mobi_description/meshes/castor_left.stl" scale="0.001 0.001 0.001"/>
-        </geometry>
-        <material name="mud_yellow"/>
-    </visual>
-    <collision>
-        <origin xyz="0.23 -0.15 -0.08" rpy="0.0 0.0 0.0"/>
-        <geometry>
-             <mesh filename="package://mobi_description/meshes/castor_left_collision.stl" scale="0.001 0.001 0.001"/>
-        </geometry>
-    </collision>
-</link>
-<joint name="left_castor_joint" type="fixed">
-    <origin xyz="-0.23 0.15 0.08" rpy="0.0 0.0 0.0"/>
-    <parent link="base_link"/>
-    <child link="left_castor_wheel"/>
-</joint>
-<link name="right_castor_wheel">
-    <inertial>
-        <origin xyz="0.23 0.15 -0.08" rpy="0.0 0.0 0.0"/>
-        <mass value="1.0"/>
-        <inertia ixx="0.1" ixy="0.0" ixz="0.0" iyy="0.1" iyz="0.0" izz="0.1"/>
-    </inertial>
-    <visual>
-        <origin xyz="0.23 0.15 -0.08" rpy="0.0 0.0 0.0"/>
-        <geometry>
-            <mesh filename="package://mobi_description/meshes/castor_right.stl" scale="0.001 0.001 0.001"/>
-        </geometry>
-        <material name="mud_yellow"/>
-    </visual>
-    <collision>
-        <origin xyz="0.23 0.15 -0.08" rpy="0.0 0.0 0.0"/>
-        <geometry>
-             <mesh filename="package://mobi_description/meshes/castor_right_collision.stl" scale="0.001 0.001 0.001"/>
-        </geometry>
-    </collision>
-</link>
-<joint name="right_castor_joint" type="fixed">
-    <origin xyz="-0.23 -0.15 0.08" rpy="0.0 0.0 0.0"/>
-    <parent link="base_link"/>
-    <child link="right_castor_wheel"/>
-</joint>
-<link name="laser_link">
-    <inertial>
-        <origin xyz="-0.154 0.0 -0.23" rpy="0.0 0.0 0.0"/>
-        <mass value="0.5"/>
-        <inertia ixx="0.1" ixy="0.0" ixz="0.0" iyy="0.1" iyz="0.0" izz="0.1"/>
-    </inertial>
-    <visual>
-        <origin xyz="-0.154 0.0 -0.23" rpy="0.0 0.0 0.0"/>
-        <geometry>
-            <mesh filename="package://mobi_description/meshes/lidar.stl" scale="0.001 0.001 0.001"/>
-        </geometry>
-        <material name="matte_brown"/>
-    </visual>
-    <collision>
-        <origin xyz="-0.154 0.0 -0.23" rpy="0.0 0.0 0.0"/>
-        <geometry>
-             <mesh filename="package://mobi_description/meshes/lidar.stl" scale="0.001 0.001 0.001"/>
-        </geometry>
-    </collision>
-</link>
-<joint name="laser_joint" type="fixed">
-    <origin xyz="0.154 0.0 0.23" rpy="0.0 0.0 0.0"/>
-    <parent link="base_link"/>
-    <child link="laser_link"/>
-</joint>
-<link name="camera_link">
-    <inertial>
-        <origin xyz="-0.276 0.0 -0.535" rpy="0.0 0.0 0.0"/>
-        <mass value="0.5"/>
-        <inertia ixx="0.1" ixy="0.0" ixz="0.0" iyy="0.1" iyz="0.0" izz="0.1"/>
-    </inertial>
-    <visual>
-        <origin xyz="-0.276 0.0 -0.535" rpy="0.0 0.0 0.0"/>
-        <geometry>
-            <mesh filename="package://mobi_description/meshes/camera.stl" scale="0.001 0.001 0.001"/>
-        </geometry>
-        <material name="matte_brown"/>
-    </visual>
-    <collision>
-        <origin xyz="-0.276 0.0 -0.535" rpy="0.0 0.0 0.0"/>
-        <geometry>
-             <mesh filename="package://mobi_description/meshes/camera.stl" scale="0.001 0.001 0.001"/>
-        </geometry>
-    </collision>
-</link>
-<joint name="camera_joint" type="fixed">
-    <origin xyz="0.276 0.0 0.535" rpy="0.0 0.0 0.0"/>
-    <parent link="base_link"/>
-    <child link="camera_link"/>
-</joint>
-<link name="camera_link_optical" />
-<joint name="camera_optical_joint" type="fixed">
-    <parent link="camera_link"/>
-    <child link="camera_link_optical"/>
-    <origin xyz="0 0 0" rpy="${-pi/2} 0 ${-pi/2}"/>
-</joint>
-<link name="imu_link">
-    <inertial>
+    <!-- Load Simulated or Real Hardware Interfaces -->
+    <xacro:arg name="is_sim" default="true"/> <!-- Getting passed as false in hardware interface launch file-->
+    <xacro:arg name="serial_port" default="/dev/ttyUSB0"/>
+    <link name="base_footprint"/>
+    <link name="base_link">
+        <inertial>
+            <origin xyz="0.0 0.0 -0.0" rpy="0.0 0.0 0.0"/>
+            <mass value="5.0"/>
+            <inertia ixx="0.1" ixy="0.0" ixz="0.0" iyy="0.1" iyz="0.0" izz="0.1"/>
+        </inertial>
+        <visual>
+            <origin xyz="0.0 0.0 -0.0" rpy="0.0 0.0 0.0"/>
+            <geometry>
+                <mesh filename="package://mobi_description/meshes/base_link.stl" scale="0.001 0.001 0.001"/>
+            </geometry>
+            <material name="silver"/>
+        </visual>
+        <collision>
+            <origin xyz="0.0 0.0 -0.0" rpy="0.0 0.0 0.0"/>
+            <geometry>
+                <mesh filename="package://mobi_description/meshes/base_link.stl" scale="0.001 0.001 0.001"/>
+            </geometry>
+        </collision>
+    </link>
+    <joint name="base_joint" type="fixed">
         <origin xyz="0.0 0.0 0.0" rpy="0.0 0.0 0.0"/>
-        <mass value="0.1"/>
-        <inertia ixx="0.1" ixy="0.0" ixz="0.0" iyy="0.1" iyz="0.0" izz="0.1"/>
-    </inertial>
-    <visual>
-        <origin xyz="0.0 0.0 0.0" rpy="0.0 0.0 0.0"/>
-        <geometry>
-            <box size="0.02 0.02 0.005"/>
-        </geometry>
-        <material name="silver"/>
-    </visual>
-    <collision>
-        <origin xyz="0.0 0.0 0.0" rpy="0.0 0.0 0.0"/>
-        <geometry>
-            <box size="0.02 0.02 0.005"/>
-        </geometry>
-    </collision>
-</link>
-<joint name="imu_joint" type="fixed">
-    <origin xyz="0.02 -0.07 0.098" rpy="0.0 0.0 0.0"/>
-    <parent link="base_link"/>
-    <child link="imu_link"/>
-</joint>
+        <parent link="base_footprint"/>
+        <child link="base_link"/>
+    </joint>
+    <link name="right_wheel">
+        <inertial>
+            <origin xyz="-0.17 0.175 -0.06" rpy="0.0 0.0 0.0"/>
+            <mass value="1.0"/>
+            <inertia ixx="0.1" ixy="0.0" ixz="0.0" iyy="0.1" iyz="0.0" izz="0.1"/>
+        </inertial>
+        <visual>
+            <origin xyz="-0.17 0.175 -0.06" rpy="0.0 0.0 0.0"/>
+            <geometry>
+                <mesh filename="package://mobi_description/meshes/right_wheel.stl" scale="0.001 0.001 0.001"/>
+            </geometry>
+            <material name="mud_yellow"/>
+        </visual>
+        <collision>
+            <origin xyz="-0.17 0.175 -0.06" rpy="0.0 0.0 0.0"/>
+            <geometry>
+                <mesh filename="package://mobi_description/meshes/right_wheel.stl" scale="0.001 0.001 0.001"/>
+            </geometry>
+        </collision>
+    </link>
+    <joint name="right_wheel_joint" type="continuous">
+        <origin xyz="0.17 -0.175 0.06" rpy="0.0 0.0 0.0"/>
+        <parent link="base_link"/>
+        <child link="right_wheel"/>
+        <axis xyz="-0.0 1.0 0.0"/>
+    </joint>
+    <link name="left_wheel">
+        <inertial>
+            <origin xyz="-0.169 -0.175 -0.059" rpy="0.0 0.0 0.0"/>
+            <mass value="1.0"/>
+            <inertia ixx="0.1" ixy="0.0" ixz="0.0" iyy="0.1" iyz="0.0" izz="0.1"/>
+        </inertial>
+        <visual>
+            <origin xyz="-0.169 -0.175 -0.059" rpy="0.0 0.0 0.0"/>
+            <geometry>
+                <mesh filename="package://mobi_description/meshes/left_wheel.stl" scale="0.001 0.001 0.001"/>
+            </geometry>
+            <material name="mud_yellow"/>
+        </visual>
+        <collision>
+            <origin xyz="-0.169 -0.175 -0.059" rpy="0.0 0.0 0.0"/>
+            <geometry>
+                <mesh filename="package://mobi_description/meshes/left_wheel.stl" scale="0.001 0.001 0.001"/>
+            </geometry>
+        </collision>
+    </link>
+    <joint name="left_wheel_joint" type="continuous">
+        <origin xyz="0.169 0.175 0.059" rpy="0.0 0.0 0.0"/>
+        <parent link="base_link"/>
+        <child link="left_wheel"/>
+        <axis xyz="-0.0 1.0 0.0"/>
+    </joint>
+    <link name="left_castor_wheel">
+        <inertial>
+            <origin xyz="0.23 -0.15 -0.08" rpy="0.0 0.0 0.0"/>
+            <mass value="1.0"/>
+            <inertia ixx="0.1" ixy="0.0" ixz="0.0" iyy="0.1" iyz="0.0" izz="0.1"/>
+        </inertial>
+        <visual>
+            <origin xyz="0.23 -0.15 -0.08" rpy="0.0 0.0 0.0"/>
+            <geometry>
+                <mesh filename="package://mobi_description/meshes/castor_left.stl" scale="0.001 0.001 0.001"/>
+            </geometry>
+            <material name="mud_yellow"/>
+        </visual>
+        <collision>
+            <origin xyz="0.23 -0.15 -0.08" rpy="0.0 0.0 0.0"/>
+            <geometry>
+                <mesh filename="package://mobi_description/meshes/castor_left_collision.stl" scale="0.001 0.001 0.001"/>
+            </geometry>
+        </collision>
+    </link>
+    <joint name="left_castor_joint" type="fixed">
+        <origin xyz="-0.23 0.15 0.08" rpy="0.0 0.0 0.0"/>
+        <parent link="base_link"/>
+        <child link="left_castor_wheel"/>
+    </joint>
+    <link name="right_castor_wheel">
+        <inertial>
+            <origin xyz="0.23 0.15 -0.08" rpy="0.0 0.0 0.0"/>
+            <mass value="1.0"/>
+            <inertia ixx="0.1" ixy="0.0" ixz="0.0" iyy="0.1" iyz="0.0" izz="0.1"/>
+        </inertial>
+        <visual>
+            <origin xyz="0.23 0.15 -0.08" rpy="0.0 0.0 0.0"/>
+            <geometry>
+                <mesh filename="package://mobi_description/meshes/castor_right.stl" scale="0.001 0.001 0.001"/>
+            </geometry>
+            <material name="mud_yellow"/>
+        </visual>
+        <collision>
+            <origin xyz="0.23 0.15 -0.08" rpy="0.0 0.0 0.0"/>
+            <geometry>
+                <mesh filename="package://mobi_description/meshes/castor_right_collision.stl" scale="0.001 0.001 0.001"/>
+            </geometry>
+        </collision>
+    </link>
+    <joint name="right_castor_joint" type="fixed">
+        <origin xyz="-0.23 -0.15 0.08" rpy="0.0 0.0 0.0"/>
+        <parent link="base_link"/>
+        <child link="right_castor_wheel"/>
+    </joint>
 </robot>
