Commit message: simulation added

File: mobi_description/urdf/gazebo.xacro (robot description, xacro)
@@ -2,20 +2,4 @@
 <robot name="mobi" xmlns:xacro="http://www.ros.org/wiki/xacro" >
     <!-- Mobi Wheels -->
-    <gazebo reference="left_castor_wheel">
-        <mu1>0.1</mu1>
-        <mu2>0.1</mu2>
-        <kp>1000000.0</kp>
-        <kd>100.0</kd>
-        <minDepth>0.001</minDepth>
-        <maxVel>1.0</maxVel>
-    </gazebo>
-    <gazebo reference="right_castor_wheel">
-        <mu1>0.1</mu1>
-        <mu2>0.1</mu2>
-        <kp>1000000.0</kp>
-        <kd>100.0</kd>
-        <minDepth>0.001</minDepth>
-        <maxVel>1.0</maxVel>
-    </gazebo>
     <gazebo reference="right_wheel">
         <mu1>1000000000000000.0</mu1>
@@ -36,4 +20,21 @@
         <fdir1>1 0 0</fdir1>
     </gazebo>
+    <!-- Caster Wheels -->
+    <gazebo reference="left_castor_wheel">
+        <mu1>0.1</mu1>
+        <mu2>0.1</mu2>
+        <!-- <kp>1000000.0</kp>
+        <kd>100.0</kd>
+        <minDepth>0.001</minDepth>
+        <maxVel>1.0</maxVel> -->
+    </gazebo>
+    <gazebo reference="right_castor_wheel">
+        <mu1>0.1</mu1>
+        <mu2>0.1</mu2>
+        <!-- <kp>1000000.0</kp>
+        <kd>100.0</kd>
+        <minDepth>0.001</minDepth>
+        <maxVel>1.0</maxVel> -->
+    </gazebo>
     <!-- ROS 2 Control -->
     <gazebo>
@@ -48,4 +49,5 @@
     </gazebo>
     <!-- Mobi Sensors -->
+    <!-- IMU -->
     <gazebo reference="imu_link">
         <sensor name="imu" type="imu">
@@ -98,7 +100,8 @@
         </sensor>
     </gazebo>
+    <!-- 2D Laser Sensor -->
     <gazebo reference="laser_link">
         <sensor name="lidar" type="gpu_lidar">
-            <pose>0 0 0 0 0 3.14</pose>
+            <pose>0 0 0 0 0 3.14</pose> <!-- Verify, if doesnot work then change-->
             <always_on>true</always_on>
             <visualize>true</visualize>
@@ -128,4 +131,5 @@
         </sensor>
     </gazebo>
+    <!-- Camera Sensor -->
     <gazebo reference="camera_link">
         <sensor name="camera" type="camera">

File: mobi_description/urdf/mobi_base.xacro (robot description, xacro)
@@ -2,5 +2,6 @@
 <robot name="mobi" xmlns:xacro="http://www.ros.org/wiki/xacro">
 <!-- Load Simulated or Real Hardware Interfaces -->
-<xacro:arg name="is_sim" default="false"/>
+<xacro:arg name="is_sim" default="true"/> <!-- Getting passed as false in hardware interface launch file-->
+<xacro:arg name="serial_port" default="/dev/ttyUSB0"/>
 <link name="base_footprint"/>
 <link name="base_link">
@@ -95,5 +96,5 @@
     </visual>
     <collision>
-        <origin xyz="0.23 -0.25 -0.08" rpy="0.0 0.0 0.0"/>
+        <origin xyz="0.23 -0.15 -0.08" rpy="0.0 0.0 0.0"/>
         <geometry>
              <mesh filename="package://mobi_description/meshes/castor_left_collision.stl" scale="0.001 0.001 0.001"/>
@@ -120,5 +121,5 @@
     </visual>
     <collision>
-        <origin xyz="0.23 0.15 -0.0" rpy="0.0 0.0 0.0"/>
+        <origin xyz="0.23 0.15 -0.08" rpy="0.0 0.0 0.0"/>
         <geometry>
              <mesh filename="package://mobi_description/meshes/castor_right_collision.stl" scale="0.001 0.001 0.001"/>
@@ -133,10 +134,10 @@
 <link name="laser_link">
     <inertial>
-        <origin xyz="-0.154 0.0 -0.19" rpy="0.0 0.0 0.0"/>
+        <origin xyz="-0.154 0.0 -0.23" rpy="0.0 0.0 0.0"/>
         <mass value="0.5"/>
         <inertia ixx="0.1" ixy="0.0" ixz="0.0" iyy="0.1" iyz="0.0" izz="0.1"/>
     </inertial>
     <visual>
-        <origin xyz="-0.154 0.0 -0.19" rpy="0.0 0.0 0.0"/>
+        <origin xyz="-0.154 0.0 -0.23" rpy="0.0 0.0 0.0"/>
         <geometry>
             <mesh filename="package://mobi_description/meshes/lidar.stl" scale="0.001 0.001 0.001"/>
@@ -145,5 +146,5 @@
     </visual>
     <collision>
-        <origin xyz="-0.154 0.0 -0.19" rpy="0.0 0.0 0.0"/>
+        <origin xyz="-0.154 0.0 -0.23" rpy="0.0 0.0 0.0"/>
         <geometry>
              <mesh filename="package://mobi_description/meshes/lidar.stl" scale="0.001 0.001 0.001"/>
@@ -152,5 +153,5 @@
 </link>
 <joint name="laser_joint" type="fixed">
-    <origin xyz="0.154 0.0 0.19" rpy="0.0 0.0 0.0"/>
+    <origin xyz="0.154 0.0 0.23" rpy="0.0 0.0 0.0"/>
     <parent link="base_link"/>
     <child link="laser_link"/>

File: mobi_description/urdf/ros2_control.xacro (robot description, xacro)
@@ -12,6 +12,12 @@
         <xacro:unless value="$(arg is_sim)">
             <hardware>
-                <plugin>mobi_firmware/MobiInterface</plugin>
-                <param name="port">/dev/ttyUSB1</param>
+                <xacro:if value="${serial_port == '/dev/ttyUSB0'}">
+                    <plugin>mobi_firmware/MobiInterface</plugin>
+                    <param name="port">/dev/ttyUSB1</param>
+                </xacro:if>
+                <xacro:if value="${serial_port == '/dev/ttyUSB1'}">
+                    <plugin>mobi_firmware/MobiInterface</plugin>
+                    <param name="port">/dev/ttyUSB0</param>
+                </xacro:if>
             </hardware>
         </xacro:unless>

Commit message: Vision Based Movement Added For Neck

File: mobi_description/urdf/gazebo.xacro (robot description, xacro)
@@ -24,16 +24,16 @@
         <mu1>0.1</mu1>
         <mu2>0.1</mu2>
-        <!-- <kp>1000000.0</kp>
+        <kp>1000000.0</kp>
         <kd>100.0</kd>
         <minDepth>0.001</minDepth>
-        <maxVel>1.0</maxVel> -->
+        <maxVel>1.0</maxVel>
     </gazebo>
     <gazebo reference="right_castor_wheel">
         <mu1>0.1</mu1>
         <mu2>0.1</mu2>
-        <!-- <kp>1000000.0</kp>
+        <kp>1000000.0</kp>
         <kd>100.0</kd>
         <minDepth>0.001</minDepth>
-        <maxVel>1.0</maxVel> -->
+        <maxVel>1.0</maxVel>
     </gazebo>
     <!-- ROS 2 Control -->

File: mobi_description/urdf/mobi_base.xacro (robot description, xacro)
@@ -44,7 +44,8 @@
         </visual>
         <collision>
-            <origin xyz="-0.17 0.175 -0.06" rpy="0.0 0.0 0.0"/>
+            <origin xyz="-0.0 0.0 -0.0" rpy="0.0 0.0 0.0"/>
             <geometry>
-                <mesh filename="package://mobi_description/meshes/right_wheel.stl" scale="0.001 0.001 0.001"/>
+                <!-- <mesh filename="package://mobi_description/meshes/right_wheel.stl" scale="0.001 0.001 0.001"/> -->
+                <sphere radius="0.06"/>
             </geometry>
         </collision>
@@ -70,7 +71,8 @@
         </visual>
         <collision>
-            <origin xyz="-0.169 -0.175 -0.059" rpy="0.0 0.0 0.0"/>
+            <origin xyz="-0.0 -0.0 -0.0" rpy="0.0 0.0 0.0"/>
             <geometry>
-                <mesh filename="package://mobi_description/meshes/left_wheel.stl" scale="0.001 0.001 0.001"/>
+                <!-- <mesh filename="package://mobi_description/meshes/left_wheel.stl" scale="0.001 0.001 0.001"/> -->
+                <sphere radius="0.06"/>
             </geometry>
         </collision>
@@ -96,7 +98,8 @@
         </visual>
         <collision>
-            <origin xyz="0.23 -0.15 -0.08" rpy="0.0 0.0 0.0"/>
+            <origin xyz="-0.0 0.0 -0.03" rpy="0.0 0.0 0.0"/>
             <geometry>
-                <mesh filename="package://mobi_description/meshes/castor_left_collision.stl" scale="0.001 0.001 0.001"/>
+                <!-- <mesh filename="package://mobi_description/meshes/castor_left_collision.stl" scale="0.001 0.001 0.001"/> -->
+                <sphere radius="0.05"/>
             </geometry>
         </collision>
@@ -121,7 +124,8 @@
         </visual>
         <collision>
-            <origin xyz="0.23 0.15 -0.08" rpy="0.0 0.0 0.0"/>
+            <origin xyz="-0.0 -0.0 -0.03" rpy="0.0 0.0 0.0"/>
             <geometry>
-                <mesh filename="package://mobi_description/meshes/castor_right_collision.stl" scale="0.001 0.001 0.001"/>
+                <!-- <mesh filename="package://mobi_description/meshes/castor_right_collision.stl" scale="0.001 0.001 0.001"/> -->
+                <sphere radius="0.05"/>
             </geometry>
         </collision>

File: mobi_description/urdf/mobi_head.xacro (robot description, xacro)
@@ -4,5 +4,5 @@
         <inertial>
             <origin xyz="-0.0054 0.0 -0.92" rpy="0.0 0.0 0.0"/>
-            <mass value="1.0"/>
+            <mass value="0.1"/>
             <inertia ixx="0.1" ixy="0.0" ixz="0.0" iyy="0.1" iyz="0.0" izz="0.1"/>
         </inertial>
@@ -31,5 +31,5 @@
         <inertial>
             <origin xyz="-0.0046 0.0 -0.96" rpy="0.0 0.0 0.0"/>
-            <mass value="1.0"/>
+            <mass value="0.1"/>
             <inertia ixx="0.1" ixy="0.0" ixz="0.0" iyy="0.1" iyz="0.0" izz="0.1"/>
         </inertial>
@@ -58,5 +58,5 @@
         <inertial>
             <origin xyz="-0.092 0.0 -0.96" rpy="0.0 0.0 0.0"/>
-            <mass value="1.0"/>
+            <mass value="0.5"/>
             <inertia ixx="0.1" ixy="0.0" ixz="0.0" iyy="0.1" iyz="0.0" izz="0.1"/>
         </inertial>
@@ -69,7 +69,8 @@
         </visual>
         <collision>
-            <origin xyz="-0.092 0.0 -0.96" rpy="0.0 0.0 0.0"/>
+            <origin xyz="-0.0 0.0 0.06" rpy="0.0 0.0 0.0"/>
             <geometry>
-                <mesh filename="package://mobi_description/meshes/head.stl" scale="0.001 0.001 0.001"/>
+                <!-- <mesh filename="package://mobi_description/meshes/head.stl" scale="0.001 0.001 0.001"/> -->
+                <box size="0.1 0.1 0.1"/>
             </geometry>
         </collision>

File: mobi_description/urdf/mobi_rail.xacro (robot description, xacro)
@@ -4,5 +4,5 @@
         <inertial>
             <origin xyz="0.06 0.0 -0.04" rpy="0.0 0.0 0.0"/>
-            <mass value="1.0"/>
+            <mass value="2.0"/>
             <inertia ixx="0.1" ixy="0.0" ixz="0.0" iyy="0.1" iyz="0.0" izz="0.1"/>
         </inertial>
@@ -15,7 +15,7 @@
         </visual>
         <collision>
-            <origin xyz="0.06 0.0 -0.04" rpy="0.0 0.0 0.0"/> <!--same as joint origin-->
+            <origin xyz="-0.05 0.0 0.5" rpy="0.0 0.0 0.0"/>
             <geometry>
-                <box size="0.05 0.15 0.8"/>
+                <box size="0.05 0.15 0.9"/>
             </geometry>
         </collision>
@@ -40,7 +40,7 @@
         </visual>
         <collision>
-            <origin xyz="0.0 0 -0.85" rpy="0.0 0.0 0.0"/>
+            <origin xyz="0.09 0 -0.05" rpy="0.0 0.0 0.0"/>
             <geometry>
-                <box size="0.2 0.3 0.4"/>
+                <box size="0.2 0.3 0.3"/>
             </geometry>
         </collision>
@@ -51,5 +51,5 @@
         <origin xyz="-0.0 0 0.85" rpy="0.0 0.0 0.0"/>
         <axis xyz="0 0 1"/>
-        <limit lower="-0.315" upper="0.0" effort="30.0" velocity="10.0"/>
+        <limit lower="-0.350" upper="0.0" effort="30.0" velocity="10.0"/>
     </joint>
 </robot>

File: mobi_description/urdf/mobi_sensors.xacro (robot description, xacro)
@@ -40,5 +40,5 @@
         </visual>
         <collision>
-            <origin xyz="-0.15 0 -0.875" rpy="0.0 0.0 0.0"/>
+            <origin xyz="0.0 0 -0.0" rpy="0.0 0.0 0.0"/>
             <geometry>
                 <box size="0.05 0.04 0.03"/>

File: mobi_description/urdf/ros2_control.xacro (robot description, xacro)
@@ -23,8 +23,9 @@
         </xacro:unless>
         <!-- ros2_control Common Interfaces -->
+         <!-- 60rpm = 6.3rad/sec-->
         <joint name="right_wheel_joint">
             <command_interface name="velocity">
-              <param name="min">-1</param>
-              <param name="max">1</param>
+                <param name="min">-6.3</param>
+                <param name="max">6.3</param>
             </command_interface>
             <state_interface name="position" />
@@ -33,10 +34,32 @@
         <joint name="left_wheel_joint">
             <command_interface name="velocity">
-              <param name="min">-1</param>
-              <param name="max">1</param>
+                <param name="min">-6.3</param>
+                <param name="max">6.3</param>
             </command_interface>
             <state_interface name="position" />
             <state_interface name="velocity" />
         </joint>
+        <!-- Make Changes Here also According to Joint Limits set in URDF-->
+        <joint name="joint_1">
+            <command_interface name="position">
+            <param name="min">-0.350</param>
+            <param name="max">0.0</param>
+            </command_interface>
+            <state_interface name="position"/>
+        </joint>
+        <joint name="joint_2">
+            <command_interface name="position">
+            <param name="min">-1.0</param>
+            <param name="max">1.0</param>
+            </command_interface>
+            <state_interface name="position"/>
+        </joint>
+        <joint name="joint_3">
+            <command_interface name="position">
+            <param name="min">-0.535</param>
+            <param name="max">0.400</param>
+            </command_interface>
+            <state_interface name="position"/>
+        </joint>
     </ros2_control>
 </robot>
