Commit message: Wheel Position Corrected in URDF and Design

File: mobi_description/urdf/gazebo.xacro (robot description, xacro)
@@ -21,5 +21,5 @@
     </gazebo>
     <!-- Caster Wheels -->
-    <gazebo reference="front_left_castor_wheel">
+    <gazebo reference="front_castor_wheel">
         <mu1>0.1</mu1>
         <mu2>0.1</mu2>
@@ -29,5 +29,5 @@
         <maxVel>1.0</maxVel>
     </gazebo>
-    <gazebo reference="front_right_castor_wheel">
+    <gazebo reference="right_castor_wheel">
         <mu1>0.1</mu1>
         <mu2>0.1</mu2>
@@ -37,13 +37,5 @@
         <maxVel>1.0</maxVel>
     </gazebo>
-    <gazebo reference="back_left_castor_wheel">
-        <mu1>0.1</mu1>
-        <mu2>0.1</mu2>
-        <kp>1000000.0</kp>
-        <kd>100.0</kd>
-        <minDepth>0.001</minDepth>
-        <maxVel>1.0</maxVel>
-    </gazebo>
-    <gazebo reference="back_right_castor_wheel">
+    <gazebo reference="left_castor_wheel">
         <mu1>0.1</mu1>
         <mu2>0.1</mu2>

File: mobi_description/urdf/mobi_base.xacro (robot description, xacro)
@@ -7,10 +7,10 @@
     <link name="base_link">
         <inertial>
-            <origin xyz="0.0 0.0 -0.0" rpy="0.0 0.0 0.0"/>
+            <origin xyz="0.0 0.0 0.0" rpy="0.0 0.0 0.0"/>
             <mass value="5.0"/>
             <inertia ixx="0.1" ixy="0.0" ixz="0.0" iyy="0.1" iyz="0.0" izz="0.1"/>
         </inertial>
         <visual>
-            <origin xyz="0.0 0.0 -0.0" rpy="0.0 0.0 0.0"/>
+            <origin xyz="0.0 0.0 0.0" rpy="0.0 0.0 0.0"/>
             <geometry>
                 <mesh filename="package://mobi_description/meshes/base_link.stl" scale="0.001 0.001 0.001"/>
@@ -32,10 +32,10 @@
     <link name="right_wheel">
         <inertial>
-            <origin xyz="-0.0 0.2275 -0.06" rpy="0.0 0.0 0.0"/>
+            <origin xyz="0.0 0.2275 -0.06" rpy="0.0 0.0 0.0"/>
             <mass value="1.0"/>
             <inertia ixx="0.1" ixy="0.0" ixz="0.0" iyy="0.1" iyz="0.0" izz="0.1"/>
         </inertial>
         <visual>
-            <origin xyz="-0.0 0.2275 -0.06" rpy="0.0 0.0 0.0"/>
+            <origin xyz="0.0 0.2275 -0.06" rpy="0.0 0.0 0.0"/>
             <geometry>
                 <mesh filename="package://mobi_description/meshes/right_wheel.stl" scale="0.001 0.001 0.001"/>
@@ -59,10 +59,10 @@
     <link name="left_wheel">
         <inertial>
-            <origin xyz="-0.0 -0.2275 -0.06" rpy="0.0 0.0 0.0"/>
+            <origin xyz="0.0 -0.2275 -0.06" rpy="0.0 0.0 0.0"/>
             <mass value="1.0"/>
             <inertia ixx="0.1" ixy="0.0" ixz="0.0" iyy="0.1" iyz="0.0" izz="0.1"/>
         </inertial>
         <visual>
-            <origin xyz="-0.0 -0.2275 -0.06" rpy="0.0 0.0 0.0"/>
+            <origin xyz="0.0 -0.2275 -0.06" rpy="0.0 0.0 0.0"/>
             <geometry>
                 <mesh filename="package://mobi_description/meshes/left_wheel.stl" scale="0.001 0.001 0.001"/>
@@ -84,107 +84,78 @@
         <axis xyz="0.0 1.0 0.0"/>
     </joint>
-    <link name="front_left_castor_wheel">
+    <link name="left_castor_wheel">
         <inertial>
-            <origin xyz="-0.22 -0.24 -0.08" rpy="0.0 0.0 0.0"/>
-            <mass value="1.0"/>
+            <origin xyz="0.355 -0.15 -0.045" rpy="0.0 0.0 0.0"/>
+            <mass value="2.0"/>
             <inertia ixx="0.1" ixy="0.0" ixz="0.0" iyy="0.1" iyz="0.0" izz="0.1"/>
         </inertial>
         <visual>
-            <origin xyz="-0.22 -0.24 -0.08" rpy="0.0 0.0 0.0"/>
+            <origin xyz="0.355 -0.15 -0.045" rpy="0.0 0.0 0.0"/>
             <geometry>
-                <mesh filename="package://mobi_description/meshes/fl_castor.stl" scale="0.001 0.001 0.001"/>
+                <mesh filename="package://mobi_description/meshes/left_castor.stl" scale="0.001 0.001 0.001"/>
             </geometry>
             <material name="mud_yellow"/>
         </visual>
         <collision>
-            <origin xyz="0.0 0.0 -0.03" rpy="0.0 0.0 0.0"/>
+            <origin xyz="0.0 0.0 -0.0" rpy="0.0 0.0 0.0"/>
             <geometry>
-                <!-- <mesh filename="package://mobi_description/meshes/castor_left_collision.stl" scale="0.001 0.001 0.001"/> -->
+                <sphere radius="0.045"/>
+            </geometry>
+        </collision>
+    </link>
+    <joint name="left_castor_joint" type="fixed">
+        <origin xyz="-0.355 0.15 0.05" rpy="0.0 0.0 0.0"/>
+        <parent link="base_link"/>
+        <child link="left_castor_wheel"/>
+    </joint>
+    <link name="right_castor_wheel">
+        <inertial>
+            <origin xyz="0.355 0.15 -0.045" rpy="0.0 0.0 0.0"/>
+            <mass value="2.0"/>
+            <inertia ixx="0.1" ixy="0.0" ixz="0.0" iyy="0.1" iyz="0.0" izz="0.1"/>
+        </inertial>
+        <visual>
+            <origin xyz="0.355 0.15 -0.045" rpy="0.0 0.0 0.0"/>
+            <geometry>
+                <mesh filename="package://mobi_description/meshes/right_castor.stl" scale="0.001 0.001 0.001"/>
+            </geometry>
+            <material name="mud_yellow"/>
+        </visual>
+        <collision>
+            <origin xyz="0.0 0.0 -0.0" rpy="0.0 0.0 0.0"/>
+            <geometry>
                 <sphere radius="0.05"/>
             </geometry>
         </collision>
     </link>
-    <joint name="front_left_castor_joint" type="fixed">
-        <origin xyz="0.22 0.24 0.08" rpy="0.0 0.0 0.0"/>
+    <joint name="right_castor_joint" type="fixed">
+        <origin xyz="-0.355 -0.15 0.045" rpy="0.0 0.0 0.0"/>
         <parent link="base_link"/>
-        <child link="front_left_castor_wheel"/>
+        <child link="right_castor_wheel"/>
     </joint>
-    <link name="front_right_castor_wheel">
+    <link name="front_castor_wheel">
         <inertial>
-            <origin xyz="-0.22 0.24 -0.08" rpy="0.0 0.0 0.0"/>
-            <mass value="1.0"/>
+            <origin xyz="0.0 0.0 -0.0" rpy="0.0 0.0 0.0"/>
+            <mass value="0.1"/>
             <inertia ixx="0.1" ixy="0.0" ixz="0.0" iyy="0.1" iyz="0.0" izz="0.1"/>
         </inertial>
         <visual>
-            <origin xyz="-0.22 0.24 -0.08" rpy="0.0 0.0 0.0"/>
+            <origin xyz="-0.1 0.0 -0.062" rpy="0.0 0.0 0.0"/>
             <geometry>
-                <mesh filename="package://mobi_description/meshes/fr_castor.stl" scale="0.001 0.001 0.001"/>
+                <mesh filename="package://mobi_description/meshes/front_castor.stl" scale="0.001 0.001 0.001"/>
             </geometry>
             <material name="mud_yellow"/>
         </visual>
         <collision>
-            <origin xyz="0.0 0.0 -0.03" rpy="0.0 0.0 0.0"/>
+            <origin xyz="0.0 0.0 -0.0" rpy="0.0 0.0 0.0"/>
             <geometry>
-                <!-- <mesh filename="package://mobi_description/meshes/castor_right_collision.stl" scale="0.001 0.001 0.001"/> -->
-                <sphere radius="0.05"/>
+                <sphere radius="0.06"/>
             </geometry>
         </collision>
     </link>
-    <joint name="front_right_castor_joint" type="fixed">
-        <origin xyz="0.22 -0.24 0.08" rpy="0.0 0.0 0.0"/>
+    <joint name="front_castor_joint" type="fixed">
+        <origin xyz="0.1 0.0 0.062" rpy="0.0 0.0 0.0"/>
         <parent link="base_link"/>
-        <child link="front_right_castor_wheel"/>
-    </joint>
-    <link name="back_left_castor_wheel">
-        <inertial>
-            <origin xyz="0.22 -0.24 -0.08" rpy="0.0 0.0 0.0"/>
-            <mass value="1.0"/>
-            <inertia ixx="0.1" ixy="0.0" ixz="0.0" iyy="0.1" iyz="0.0" izz="0.1"/>
-        </inertial>
-        <visual>
-            <origin xyz="0.22 -0.24 -0.08" rpy="0.0 0.0 0.0"/>
-            <geometry>
-                <mesh filename="package://mobi_description/meshes/bl_castor.stl" scale="0.001 0.001 0.001"/>
-            </geometry>
-            <material name="mud_yellow"/>
-        </visual>
-        <collision>
-            <origin xyz="0.0 0.0 -0.03" rpy="0.0 0.0 0.0"/>
-            <geometry>
-                <!-- <mesh filename="package://mobi_description/meshes/castor_left_collision.stl" scale="0.001 0.001 0.001"/> -->
-                <sphere radius="0.05"/>
-            </geometry>
-        </collision>
-    </link>
-    <joint name="back_left_castor_joint" type="fixed">
-        <origin xyz="-0.22 0.24 0.08" rpy="0.0 0.0 0.0"/>
-        <parent link="base_link"/>
-        <child link="back_left_castor_wheel"/>
-    </joint>
-    <link name="back_right_castor_wheel">
-        <inertial>
-            <origin xyz="0.22 0.24 -0.08" rpy="0.0 0.0 0.0"/>
-            <mass value="1.0"/>
-            <inertia ixx="0.1" ixy="0.0" ixz="0.0" iyy="0.1" iyz="0.0" izz="0.1"/>
-        </inertial>
-        <visual>
-            <origin xyz="0.22 0.24 -0.08" rpy="0.0 0.0 0.0"/>
-            <geometry>
-                <mesh filename="package://mobi_description/meshes/br_castor.stl" scale="0.001 0.001 0.001"/>
-            </geometry>
-            <material name="mud_yellow"/>
-        </visual>
-        <collision>
-            <origin xyz="0.0 0.0 -0.03" rpy="0.0 0.0 0.0"/>
-            <geometry>
-                <!-- <mesh filename="package://mobi_description/meshes/castor_right_collision.stl" scale="0.001 0.001 0.001"/> -->
-                <sphere radius="0.05"/>
-            </geometry>
-        </collision>
-    </link>
-    <joint name="back_right_castor_joint" type="fixed">
-        <origin xyz="-0.22 -0.24 0.08" rpy="0.0 0.0 0.0"/>
-        <parent link="base_link"/>
-        <child link="back_right_castor_wheel"/>
+        <child link="front_castor_wheel"/>
     </joint>
 </robot>

File: mobi_description/urdf/mobi_sensors.xacro (robot description, xacro)
@@ -3,10 +3,10 @@
     <link name="laser_link">
         <inertial>
-            <origin xyz="0.013 0.0 -0.23" rpy="0.0 0.0 0.0"/>
+            <origin xyz="0.015 0.0 -0.23" rpy="0.0 0.0 0.0"/>
             <mass value="0.5"/>
             <inertia ixx="0.1" ixy="0.0" ixz="0.0" iyy="0.1" iyz="0.0" izz="0.1"/>
         </inertial>
         <visual>
-            <origin xyz="0.013 0.0 -0.23" rpy="0.0 0.0 0.0"/>
+            <origin xyz="0.015 0.0 -0.23" rpy="0.0 0.0 0.0"/>
             <geometry>
                 <mesh filename="package://mobi_description/meshes/lidar.stl" scale="0.001 0.001 0.001"/>
@@ -15,5 +15,5 @@
         </visual>
         <collision>
-            <origin xyz="0.013 0.0 -0.23" rpy="0.0 0.0 0.0"/>
+            <origin xyz="0.015 0.0 -0.23" rpy="0.0 0.0 0.0"/>
             <geometry>
                 <mesh filename="package://mobi_description/meshes/lidar.stl" scale="0.001 0.001 0.001"/> <!--Kepp it as it is-->
@@ -22,5 +22,5 @@
     </link>
     <joint name="laser_joint" type="fixed">
-        <origin xyz="-0.013 0.0 0.23" rpy="0.0 0.0 0.0"/>
+        <origin xyz="-0.15 0.0 0.23" rpy="0.0 0.0 0.0"/>
         <parent link="base_link"/>
         <child link="laser_link"/>
@@ -47,5 +47,5 @@
     </link>
     <joint name="camera_joint" type="fixed">
-        <origin xyz="0.25 0.0 0.32" rpy="0.0 0.0 0.0"/>
+        <origin xyz="0.108 0.0 0.32" rpy="0.0 0.0 0.0"/>
         <parent link="base_link"/>
         <child link="camera_link"/>
@@ -84,10 +84,10 @@
     <link name="ultrasonic_link">
         <inertial>
-            <origin xyz="-0.22 0.0 -0.12" rpy="0.0 0.0 0.0"/>
+            <origin xyz="-0.25 0.0 -0.12" rpy="0.0 0.0 0.0"/>
             <mass value="0.1"/>
             <inertia ixx="0.1" ixy="0.0" ixz="0.0" iyy="0.1" iyz="0.0" izz="0.1"/>
         </inertial>
         <visual>
-            <origin xyz="-0.22 0.0 -0.12" rpy="0.0 0.0 0.0"/>
+            <origin xyz="-0.25 0.0 -0.12" rpy="0.0 0.0 0.0"/>
             <geometry>
                 <mesh filename="package://mobi_description/meshes/ultrasonic.stl" scale="0.001 0.001 0.001"/>
@@ -96,5 +96,5 @@
         </visual>
         <collision>
-            <origin xyz="-0.22 0.0 -0.12" rpy="0.0 0.0 0.0"/>
+            <origin xyz="-0.25 0.0 -0.12" rpy="0.0 0.0 0.0"/>
             <geometry>
                 <mesh filename="package://mobi_description/meshes/ultrasonic.stl" scale="0.001 0.001 0.001"/>
@@ -103,5 +103,5 @@
     </link>
     <joint name="ultrasonic_joint" type="fixed">
-        <origin xyz="0.22 0.0 0.12" rpy="0.0 0.0 0.0"/>
+        <origin xyz="0.105 0.0 0.12" rpy="0.0 0.0 0.0"/>
         <parent link="base_link"/>
         <child link="ultrasonic_link"/>
