Commit message: simulation nav2 added

File: mobi_description/urdf/mobi_base.xacro (robot description, xacro)
@@ -12,5 +12,5 @@
         </inertial>
         <visual>
-            <origin xyz="0.0 0.0 0.0" rpy="0.0 0.0 0.0"/>
+            <origin xyz="0.15 0.0 0.0" rpy="0.0 0.0 0.0"/>
             <geometry>
                 <mesh filename="package://mobi_description/meshes/base_link.stl" scale="0.001 0.001 0.001"/>
@@ -26,5 +26,5 @@
     </link>
     <joint name="base_joint" type="fixed">
-        <origin xyz="0.0 0.0 0.0" rpy="0.0 0.0 0.0"/>
+        <origin xyz="-0.15 0.0 0.0" rpy="0.0 0.0 0.0"/>
         <parent link="base_footprint"/>
         <child link="base_link"/>
@@ -52,5 +52,5 @@
     </link>
     <joint name="right_wheel_joint" type="continuous">
-        <origin xyz="0.0 -0.2275 0.06" rpy="0.0 0.0 0.0"/>
+        <origin xyz="0.15 -0.2275 0.06" rpy="0.0 0.0 0.0"/>
         <parent link="base_link"/>
         <child link="right_wheel"/>
@@ -79,5 +79,5 @@
     </link>
     <joint name="left_wheel_joint" type="continuous">
-        <origin xyz="0.0 0.2275 0.06" rpy="0.0 0.0 0.0"/>
+        <origin xyz="0.15 0.2275 0.06" rpy="0.0 0.0 0.0"/>
         <parent link="base_link"/>
         <child link="left_wheel"/>
@@ -105,5 +105,5 @@
     </link>
     <joint name="left_castor_joint" type="fixed">
-        <origin xyz="-0.355 0.15 0.05" rpy="0.0 0.0 0.0"/>
+        <origin xyz="-0.205 0.15 0.05" rpy="0.0 0.0 0.0"/>
         <parent link="base_link"/>
         <child link="left_castor_wheel"/>
@@ -130,5 +130,5 @@
     </link>
     <joint name="right_castor_joint" type="fixed">
-        <origin xyz="-0.355 -0.15 0.045" rpy="0.0 0.0 0.0"/>
+        <origin xyz="-0.205 -0.15 0.045" rpy="0.0 0.0 0.0"/>
         <parent link="base_link"/>
         <child link="right_castor_wheel"/>
@@ -155,5 +155,5 @@
     </link>
     <joint name="front_castor_joint" type="fixed">
-        <origin xyz="0.1 0.0 0.062" rpy="0.0 0.0 0.0"/>
+        <origin xyz="0.25 0.0 0.062" rpy="0.0 0.0 0.0"/>
         <parent link="base_link"/>
         <child link="front_castor_wheel"/>

File: mobi_description/urdf/mobi_sensors.xacro (robot description, xacro)
@@ -22,5 +22,5 @@
     </link>
     <joint name="laser_joint" type="fixed">
-        <origin xyz="-0.15 0.0 0.23" rpy="0.0 0.0 0.0"/>
+        <origin xyz="0.0 0.0 0.23" rpy="0.0 0.0 0.0"/>
         <parent link="base_link"/>
         <child link="laser_link"/>
@@ -47,5 +47,5 @@
     </link>
     <joint name="camera_joint" type="fixed">
-        <origin xyz="0.108 0.0 0.32" rpy="0.0 0.0 0.0"/>
+        <origin xyz="0.258 0.0 0.32" rpy="0.0 0.0 0.0"/>
         <parent link="base_link"/>
         <child link="camera_link"/>
@@ -78,5 +78,5 @@
     </link>
     <joint name="imu_joint" type="fixed">
-        <origin xyz="0.0 0.0 0.125" rpy="0.0 0.0 0.0"/>
+        <origin xyz="0.15 0.0 0.125" rpy="0.0 0.0 0.0"/>
         <parent link="base_link"/>
         <child link="imu_link"/>
@@ -103,5 +103,5 @@
     </link>
     <joint name="ultrasonic_joint" type="fixed">
-        <origin xyz="0.105 0.0 0.12" rpy="0.0 0.0 0.0"/>
+        <origin xyz="0.255 0.0 0.12" rpy="0.0 0.0 0.0"/>
         <parent link="base_link"/>
         <child link="ultrasonic_link"/>

Commit message: Undock Working Real Robot

File: mobi_description/urdf/mobi_base.xacro (robot description, xacro)
@@ -7,5 +7,5 @@
     <link name="base_link">
         <inertial>
-            <origin xyz="0.0 0.0 0.0" rpy="0.0 0.0 0.0"/>
+            <origin xyz="0.15 0.0 0.0" rpy="0.0 0.0 0.0"/>
             <mass value="5.0"/>
             <inertia ixx="0.1" ixy="0.0" ixz="0.0" iyy="0.1" iyz="0.0" izz="0.1"/>
@@ -19,5 +19,5 @@
         </visual>
         <collision>
-            <origin xyz="0.0 0.0 0.0" rpy="0.0 0.0 0.0"/>
+            <origin xyz="0.15 0.0 0.0" rpy="0.0 0.0 0.0"/>
             <geometry>
                 <mesh filename="package://mobi_description/meshes/base_link.stl" scale="0.001 0.001 0.001"/>
@@ -29,4 +29,29 @@
         <parent link="base_footprint"/>
         <child link="base_link"/>
+    </joint>
+    <link name="torso_link">
+        <inertial>
+            <origin xyz="0.15 0.0 -0.3" rpy="0.0 0.0 0.0"/>
+            <mass value="3.0"/>
+            <inertia ixx="0.1" ixy="0.0" ixz="0.0" iyy="0.1" iyz="0.0" izz="0.1"/>
+        </inertial>
+        <visual>
+            <origin xyz="0.15 0.0 -0.3" rpy="0.0 0.0 0.0"/>
+            <geometry>
+                <mesh filename="package://mobi_description/meshes/torso.stl" scale="0.001 0.001 0.001"/>
+            </geometry>
+            <material name="silver"/>
+        </visual>
+        <collision>
+            <origin xyz="0.15 0.0 -0.3" rpy="0.0 0.0 0.0"/>
+            <geometry>
+                <mesh filename="package://mobi_description/meshes/torso.stl" scale="0.001 0.001 0.001"/>
+            </geometry>
+        </collision>
+    </link>
+    <joint name="torso_joint" type="fixed">
+        <origin xyz="-0.0 0.0 0.3" rpy="0.0 0.0 0.0"/>
+        <parent link="base_link"/>
+        <child link="torso_link"/>
     </joint>
     <link name="right_wheel">
@@ -136,5 +161,5 @@
     <link name="front_castor_wheel">
         <inertial>
-            <origin xyz="0.0 0.0 -0.0" rpy="0.0 0.0 0.0"/>
+            <origin xyz="-0.1 0.0 -0.062" rpy="0.0 0.0 0.0"/>
             <mass value="0.1"/>
             <inertia ixx="0.1" ixy="0.0" ixz="0.0" iyy="0.1" iyz="0.0" izz="0.1"/>
